Commit message: fix small bug on rigid fluid force implementation

File: data/models/Dragon_50k.urdf (robot description, URDF)
Before this commit: robot custom_mesh_robot, 1 links, 0 joints
Links:
- link baseLink: mass 118.37522888183594 -> 118.3752212524414

Commit message: test single movable rigid with dfsph

File: data/models/Dragon_50k.urdf (robot description, URDF)
Before this commit: robot custom_mesh_robot, 1 links, 0 joints
Links:
- link baseLink: mass 118.3752212524414 -> 118.37522888183594

Commit message: fix small bugs in orientation of rigid

File: data/models/Dragon_50k.urdf (robot description, URDF)
Before this commit: robot custom_mesh_robot, 1 links, 0 joints
Links:
- link baseLink: mass 118.3752212524414 -> 118.93843841552734

Commit message: readme WIP

File: data/models/Dragon_50k.urdf (robot description, URDF)
Before this commit: robot custom_mesh_robot, 1 links, 0 joints
Links:
- link baseLink: mass 118.93843841552734 -> 118.93843078613281

Commit message: enable rigid id not starting from zero

File: data/models/Dragon_50k.urdf (robot description, URDF)
Before this commit: robot custom_mesh_robot, 1 links, 0 joints
Links:
- link baseLink: mass 118.93843078613281 -> 118.93843841552734
